File: hardware/kicad/can-foc-actuator.kicad_sch (KiCad schematic)
At the start: 75 parts, among them J1 12V IN, J10 CAN OUT, J11 SWD, J12 UART, J13 12V OUT, J2 MOTOR, J3 AS5600 + NTC, J4 SPI_A motor side, J5 SPI_B output side, J6 VM to Mini, J9 CAN IN, U1 STM32G431CBT6, U2 SN65HVD230, U3 INA240A1D, U4 INA240A1D, U6 SimpleFOC Mini, U7 MP1584EN module, U8 AMS1117-3.3, Y1 8MHz

Commit message: Generate the Mini socket from its vendor board file; drop the MP1584, LDO direct
Two changes.

1. The SimpleFOC Mini is now properly part of the project rather than
   transcribed into it.  hardware/vendor/simplefocmini/ holds the module's own
   EasyEDA PCB export (MIT, byte-identical to the file supplied) plus its
   licence and a provenance note, and tools/gen_kicad.py parses it at build
   time to produce the socket footprint: H1 pads 1-10, P1 pads renumbered
   11-13 (OUT3 OUT2 OUT1), and the silkscreen/courtyard from the board-outline
   layer.  The parser reproduces the previously hand-transcribed pad table
   exactly, and additionally gives the real module edge: 23.0 x 21.0 mm running
   x -13.72..+9.29, y -1.91..+19.05 mm about H1 pad 1.  The old silkscreen was
   a pad bounding box and understated the module by 7 mm on the screw-terminal
   side, which is the clearance that matters when placing it.

2. The MP1584 is gone: the AMS1117-3.3 now runs straight off the 12 V bus.
   The itemised 3V3 load is 76 mA (MCU 30, CAN 15, 2x INA240 5, AS5600 6.5,
   joint encoder 15, LEDs and pull-ups 4), so the LDO drops 8.7 V at 76 mA =
   0.66 W and reaches Tj ~93 C at 40 C ambient even on a poor SOT-223 pour.
   U7, C23 and the +5V net are removed; C5/C21 become the LDO input
   decoupling on VBUS.

   The cost is that the AMS1117, not the DRV8313, now sets the bus ceiling:
   18 V absolute max and 1.17 W already at 15 V, so this build is 12 V only
   and the firmware over-voltage trip moves from 16 V to 15 V.  A higher bus
   needs a switching pre-regulator back in front of the LDO; the MP1584
   symbol and footprint stay in the project library, unused, for that.

design_calcs.py gains the itemised load and an LDO thermal sweep in place of
the buck maths; board_design.py, foc_config.h, the BOM/inventory/netlist CSVs,
both wiring diagrams and docs 01/02/06/07/08 and the READMEs follow.
check_design.py still passes: 51 nets, 8 no-connects, netlist matching KiCad's
own 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
Parts:
- removed C23: 100nF/250V, Capacitor_SMD:C_1206_3216Metric, symbol Device:C
- removed U7: MP1584EN module, canfoc:MP1584_Module_4pin, symbol canfoc:MP1584_Module
Connections:
- net +5V is gone; now on net VBUS: C21.1, U8.3 (VI)
Other:
- note added: "LOGIC RAIL 12 V -> AMS1117 -> 3V3 -> VDDA"
- note removed: "LOGIC RAILS 12 V -> 5 V -> 3V3 -> VDDA"
- moved on the sheet: C11, C12, C13, C21, C5, C6, C7, R23, U8
